Commit message: fix up everything and fix legs in human and classic pushup

File: atlaspushup/urdf/atlas_v5.urdf (robot description, URDF)
Before this commit: robot drc_skeleton, 45 links, 44 joints
Links:
- removed link cube
- removed link cube-xm
- removed link cube-xp
- removed link cube-ym
- removed link cube-yp
- removed link cube-zm
- removed link cube-zp
- removed link world
Joints:
- removed joint attach-cube
- removed joint attach-cube-xm
- removed joint attach-cube-xp
- removed joint attach-cube-ym
- removed joint attach-cube-yp
- removed joint attach-cube-zm
- removed joint attach-cube-zp
- removed joint theta1
